File: DRV2.kicad_sch (KiCad schematic)
At the start: 15 parts

Commit message: Motor symbol corrected, Oscillator circuitry added and external footprints added
Parts:
- removed UB: DRV10970PWPR, symbol DRV10970PWPR:DRV10970PWPR
- added UA?: DRV10970PWPR, DRV10970PWPR:SOP65P640X120-25N, symbol DRV10970PWPR:DRV10970PWPR
Connections:
- net BRK_2: now also UA?.21 (BRKMOD)
- net CMT_2: now also UA?.20 (CMTMOD)
- net CPN: now also UA?.10 (CPN)
- net CPP: now also UA?.9 (CPP)
- net CS: now also UA?.17 (CS)
- net FG_2: now also UA?.24 (FG)
- net FR_2: now also UA?.23 (FR)
- net GND: now also UA?.12 (GND), UA?.25 (EP)
- net MOT_POW: now also UA?.15 (VM)
- net MOT_PWM_2: now also UA?.19 (PWM)
- net RD_2: now also UA?.18 (RD)
- net RTRY: now also UA?.22 (RETRY)
- net U_2: now also UA?.14 (U)
- net U_HP_2: now also UA?.2 (U_HP)
- net VCP: now also UA?.8 (VCP)
- net VINT: now also UA?.16 (VINT)
- net VINT_BY_2: now also UA?.3 (U_HN), UA?.5 (V_HN), UA?.7 (W_HN)
- net V_2: now also UA?.13 (V)
- net V_HP_2: now also UA?.4 (V_HP)
- net W_2: now also UA?.11 (W)
- net W_HP_2: now also UA?.6 (W_HP)
- net at TPB1.1: now also UA?.1 (DAA)
Changed lines of the file:
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@@
   (symbol (lib_id "power:GND") (at 143.51 142.875 0) (unit 1)
     (in_bom yes) (on_board yes)
-    (property "Reference" "#PWR?" (id 0) (at 143.51 149.225 0)
+    (property "Reference" "#PWR0168" (id 0) (at 143.51 149.225 0)
       (effects (font (size 1.27 1.27)) hide)
     )
@@
     (pin "2")
   )
-  (symbol (lib_id "Device:R") (at 95.25 66.04 0) (unit 1)
-    (in_bom yes) (on_board yes) (fields_autoplaced)
-    (property "Reference" "RB2" (id 0) (at 97.79 64.7699 0)
-      (effects (font (size 1.27 1.27)) (justify left))
-    )
-    (property "Value" "4.7K" (id 1) (at 97.79 67.3099 0)
-      (effects (font (size 1.27 1.27)) (justify left))
-    )
-    (property "Footprint" "" (id 2) (at 93.472 66.04 90)
-      (effects (font (size 1.27 1.27)) hide)
-    )
-    (property "Datasheet" "~" (id 3) (at 95.25 66.04 0)
-      (effects (font (size 1.27 1.27)) hide)
-    )
-    (pin "1")
-    (pin "2")
-  )
   (symbol (lib_id "DRV10970PWPR:DRV10970PWPR") (at 127 72.39 0) (unit 1)
     (in_bom yes) (on_board yes) (fields_autoplaced)
-    (property "Reference" "UB" (id 0) (at 142.24 59.69 0))
+    (property "Reference" "UA?" (id 0) (at 142.24 59.69 0))
     (property "Value" "DRV10970PWPR" (id 1) (at 142.24 62.23 0))
-    (property "Footprint" "" (id 2) (at 127 72.39 0)
+    (property "Footprint" "DRV10970PWPR:SOP65P640X120-25N" (id 2) (at 127 72.39 0)
       (effects (font (size 1.27 1.27)) hide)
     )
@@
     (pin "9")
   )
+  (symbol (lib_id "Device:R") (at 95.25 66.04 0) (unit 1)
+    (in_bom yes) (on_board yes) (fields_autoplaced)
+    (property "Reference" "RB2" (id 0) (at 97.79 64.7699 0)
+      (effects (font (size 1.27 1.27)) (justify left))
+    )
+    (property "Value" "4.7K" (id 1) (at 97.79 67.3099 0)
+      (effects (font (size 1.27 1.27)) (justify left))
+    )
+    (property "Footprint" "" (id 2) (at 93.472 66.04 90)
+      (effects (font (size 1.27 1.27)) hide)
+    )
+    (property "Datasheet" "~" (id 3) (at 95.25 66.04 0)
+      (effects (font (size 1.27 1.27)) hide)
+    )
+    (pin "1")
+    (pin "2")
+  )
   (symbol (lib_id "Device:R") (at 194.31 93.98 0) (unit 1)
     (in_bom yes) (on_board yes) (fields_autoplaced)
@@
   (symbol (lib_id "power:GND") (at 177.8 105.41 0) (unit 1)
     (in_bom yes) (on_board yes) (fields_autoplaced)
-    (property "Reference" "#PWR?" (id 0) (at 177.8 111.76 0)
+    (property "Reference" "#PWR0170" (id 0) (at 177.8 111.76 0)
       (effects (font (size 1.27 1.27)) hide)
     )
@@
   (symbol (lib_id "power:GND") (at 142.24 113.03 0) (unit 1)
     (in_bom yes) (on_board yes) (fields_autoplaced)
-    (property "Reference" "#PWR?" (id 0) (at 142.24 119.38 0)
+    (property "Reference" "#PWR0169" (id 0) (at 142.24 119.38 0)
       (effects (font (size 1.27 1.27)) hide)
     )
@@
   (symbol (lib_id "power:GND") (at 194.31 97.79 0) (unit 1)
     (in_bom yes) (on_board yes) (fields_autoplaced)
-    (property "Reference" "#PWR?" (id 0) (at 194.31 104.14 0)
+    (property "Reference" "#PWR0171" (id 0) (at 194.31 104.14 0)
       (effects (font (size 1.27 1.27)) hide)
     )
@@
   (symbol (lib_id "power:GND") (at 127 100.33 0) (unit 1)
     (in_bom yes) (on_board yes) (fields_autoplaced)
-    (property "Reference" "#PWR?" (id 0) (at 127 106.68 0)
+    (property "Reference" "#PWR0167" (id 0) (at 127 106.68 0)
       (effects (font (size 1.27 1.27)) hide)
     )
@@
   (symbol (lib_id "power:GND") (at 212.09 135.89 0) (unit 1)
     (in_bom yes) (on_board yes) (fields_autoplaced)
-    (property "Reference" "#PWR?" (id 0) (at 212.09 142.24 0)
-      (effects (font (size 1.27 1.27)) hide)
-    )
+    (property "Reference" "#PWR0172" (id 0) (at 212.09 142.24 0)
+      (effects (font (size 1.27 1.27)) hide)
+    )

Commit message: MCU interfaces are done! Check the Changes and Complete ERC modifications
Other:
- company: (none) -> Parikshit Student Satellite Team
- title: (none) -> AOCS BOARD
Changed lines of the file:
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@@
 (kicad_sch (version 20211123) (generator eeschema)
   (paper "A4")
+  (title_block
+    (title "AOCS BOARD")
+    (company "Parikshit Student Satellite Team")
+  )
   (junction (at 172.72 62.23) (diameter 0) (color 0 0 0 0)
   )
@@
   )
   (wire (pts (xy 212.09 121.92) (xy 212.09 124.46))
+    (stroke (width 0) (type default) (color 0 0 0 0))
+  )
+  (wire (pts (xy 24.765 118.745) (xy 24.765 117.475))
     (stroke (width 0) (type default) (color 0 0 0 0))
   )
@@
     (pin "1")
     (pin "2")
+  )
+  (symbol (lib_id "power:PWR_FLAG") (at 24.765 117.475 0) (unit 1)
+    (in_bom yes) (on_board yes) (fields_autoplaced)
+    (property "Reference" "#FLG0108" (id 0) (at 24.765 115.57 0)
+      (effects (font (size 1.27 1.27)) hide)
+    )
+    (property "Value" "PWR_FLAG" (id 1) (at 24.765 111.76 0))
+    (property "Footprint" "" (id 2) (at 24.765 117.475 0)
+      (effects (font (size 1.27 1.27)) hide)
+    )
+    (property "Datasheet" "~" (id 3) (at 24.765 117.475 0)
+      (effects (font (size 1.27 1.27)) hide)
+    )
+    (pin "1")
   )
   (symbol (lib_id "DRV10970PWPR:DRV10970PWPR") (at 127 72.39 0) (unit 1)
@@
     (pin "2")
   )
+  (symbol (lib_id "power:GND") (at 24.765 118.745 0) (unit 1)
+    (in_bom yes) (on_board yes) (fields_autoplaced)
+    (property "Reference" "#PWR0272" (id 0) (at 24.765 125.095 0)
+      (effects (font (size 1.27 1.27)) hide)
+    )
+    (property "Value" "GND" (id 1) (at 24.765 123.19 0))
+    (property "Footprint" "" (id 2) (at 24.765 118.745 0)
+      (effects (font (size 1.27 1.27)) hide)
+    )
+    (property "Datasheet" "" (id 3) (at 24.765 118.745 0)
+      (effects (font (size 1.27 1.27)) hide)
+    )
+    (pin "1")
+  )
   (symbol (lib_id "power:GND") (at 177.8 105.41 0) (unit 1)

Commit message: Max ERC errors corrected
Changed lines of the file:
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@@
-    (stroke (width 0) (type default) (color 0 0 0 0))
-  )
-  (wire (pts (xy 175.26 63.5) (xy 175.26 62.23))
     (stroke (width 0) (type default) (color 0 0 0 0))
   )
@@
     (stroke (width 0) (type default) (color 0 0 0 0))
   )
-  (wire (pts (xy 24.765 118.745) (xy 24.765 117.475))
-    (stroke (width 0) (type default) (color 0 0 0 0))
-  )
   (wire (pts (xy 143.51 142.875) (xy 143.51 142.24))
     (stroke (width 0) (type default) (color 0 0 0 0))
@@
   (label "CS" (at 191.77 121.92 0)
     (effects (font (size 1.27 1.27)) (justify left bottom))
-  )
-  (global_label "MCU_POW" (shape bidirectional) (at 175.26 63.5 0) (fields_autoplaced)
-    (effects (font (size 1.27 1.27)) (justify left))
-    (property "Intersheet References" "${INTERSHEET_REFS}" (id 0) (at 186.7445 63.4206 0)
-      (effects (font (size 1.27 1.27)) (justify left) hide)
-    )
   )
   (hierarchical_label "MOT_POW" (shape bidirectional) (at 114.3 144.78 180)
@@
   )
   (hierarchical_label "MOT_POW" (shape bidirectional) (at 160.02 95.25 0)
+    (effects (font (size 1.27 1.27)) (justify left))
+  )
+  (hierarchical_label "MCU_POW" (shape bidirectional) (at 175.26 62.23 0)
     (effects (font (size 1.27 1.27)) (justify left))
   )
@@
     (pin "2")
   )
+  (symbol (lib_id "upsat-comms-hardware:GND") (at 177.8 105.41 0) (unit 1)
+    (in_bom yes) (on_board yes) (fields_autoplaced)
+    (property "Reference" "#PWR0167" (id 0) (at 177.8 111.76 0)
+      (effects (font (size 1.27 1.27)) hide)
+    )
+    (property "Value" "GND" (id 1) (at 177.8 109.855 0))
+    (property "Footprint" "" (id 2) (at 177.8 105.41 0))
+    (property "Datasheet" "" (id 3) (at 177.8 105.41 0))
+    (pin "1")
+  )
   (symbol (lib_id "Device:R") (at 110.49 66.04 0) (unit 1)
     (in_bom yes) (on_board yes) (fields_autoplaced)
@@
     (pin "2")
   )
-  (symbol (lib_id "power:GND") (at 143.51 142.875 0) (unit 1)
-    (in_bom yes) (on_board yes)
-    (property "Reference" "#PWR0168" (id 0) (at 143.51 149.225 0)
-      (effects (font (size 1.27 1.27)) hide)
-    )
-    (property "Value" "GND" (id 1) (at 147.32 144.78 0))
-    (property "Footprint" "" (id 2) (at 143.51 142.875 0)
-      (effects (font (size 1.27 1.27)) hide)
-    )
-    (property "Datasheet" "" (id 3) (at 143.51 142.875 0)
-      (effects (font (size 1.27 1.27)) hide)
-    )
-    (pin "1")
-  )
   (symbol (lib_id "Device:R") (at 172.72 78.74 0) (unit 1)
     (in_bom yes) (on_board yes) (fields_autoplaced)
@@
     (pin "2")
   )
+  (symbol (lib_id "upsat-comms-hardware:GND") (at 194.31 97.79 0) (unit 1)
+    (in_bom yes) (on_board yes) (fields_autoplaced)
+    (property "Reference" "#PWR0171" (id 0) (at 194.31 104.14 0)
+      (effects (font (size 1.27 1.27)) hide)
+    )
+    (property "Value" "GND" (id 1) (at 194.31 102.235 0))
+    (property "Footprint" "" (id 2) (at 194.31 97.79 0))
+    (property "Datasheet" "" (id 3) (at 194.31 97.79 0))
+    (pin "1")
+  )
+  (symbol (lib_id "upsat-comms-hardware:GND") (at 143.51 142.875 0) (unit 1)
+    (in_bom yes) (on_board yes) (fields_autoplaced)
+    (property "Reference" "#PWR0169" (id 0) (at 143.51 149.225 0)
+      (effects (font (size 1.27 1.27)) hide)
+    )
+    (property "Value" "GND" (id 1) (at 143.51 147.32 0))
+    (property "Footprint" "" (id 2) (at 143.51 142.875 0))
+    (property "Datasheet" "" (id 3) (at 143.51 142.875 0))
+    (pin "1")
+  )
+  (symbol (lib_id "upsat-comms-hardware:GND") (at 127 100.33 0) (unit 1)
+    (in_bom yes) (on_board yes) (fields_autoplaced)
+    (property "Reference" "#PWR0168" (id 0) (at 127 106.68 0)
+      (effects (font (size 1.27 1.27)) hide)
+    )
+    (property "Value" "GND" (id 1) (at 127 104.775 0))
+    (property "Footprint" "" (id 2) (at 127 100.33 0))
+    (property "Datasheet" "" (id 3) (at 127 100.33 0))
+    (pin "1")
+  )
+  (symbol (lib_id "upsat-comms-hardware:GND") (at 212.09 135.89 0) (unit 1)
+    (in_bom yes) (on_board yes) (fields_autoplaced)
+    (property "Reference" "#PWR0172" (id 0) (at 212.09 142.24 0)
+      (effects (font (size 1.27 1.27)) hide)
+    )
+    (property "Value" "GND" (id 1) (at 212.09 140.335 0))
+    (property "Footprint" "" (id 2) (at 212.09 135.89 0))
+    (property "Datasheet" "" (id 3) (at 212.09 135.89 0))
+    (pin "1")
+  )
   (symbol (lib_id "pspice:C") (at 128.27 135.89 0) (unit 1)
     (in_bom yes) (on_board yes) (fields_autoplaced)
@@
     (pin "1")
     (pin "2")
-  )
-  (symbol (lib_id "power:PWR_FLAG") (at 24.765 117.475 0) (unit 1)
-    (in_bom yes) (on_board yes) (fields_autoplaced)
-    (property "Reference" "#FLG0108" (id 0) (at 24.765 115.57 0)
-      (effects (font (size 1.27 1.27)) hide)
-    )
-    (property "Value" "PWR_FLAG" (id 1) (at 24.765 111.76 0))
-    (property "Footprint" "" (id 2) (at 24.765 117.475 0)
-      (effects (font (size 1.27 1.27)) hide)
-    )
-    (property "Datasheet" "~" (id 3) (at 24.765 117.475 0)
-      (effects (font (size 1.27 1.27)) hide)
-    )
-    (pin "1")
   )
   (symbol (lib_id "DRV10970PWPR:DRV10970PWPR") (at 127 72.39 0) (unit 1)
@@
     (pin "2")
   )
-  (symbol (lib_id "power:GND") (at 24.765 118.745 0) (unit 1)
-    (in_bom yes) (on_board yes) (fields_autoplaced)
-    (property "Reference" "#PWR0272" (id 0) (at 24.765 125.095 0)
-      (effects (font (size 1.27 1.27)) hide)
-    )
-    (property "Value" "GND" (id 1) (at 24.765 123.19 0))
-    (property "Footprint" "" (id 2) (at 24.765 118.745 0)
-      (effects (font (size 1.27 1.27)) hide)
-    )
-    (property "Datasheet" "" (id 3) (at 24.765 118.745 0)
-      (effects (font (size 1.27 1.27)) hide)
-    )
-    (pin "1")
-  )
-  (symbol (lib_id "power:GND") (at 177.8 105.41 0) (unit 1)
-    (in_bom yes) (on_board yes) (fields_autoplaced)
-    (property "Reference" "#PWR0170" (id 0) (at 177.8 111.76 0)
-      (effects (font (size 1.27 1.27)) hide)
-    )
-    (property "Value" "GND" (id 1) (at 177.8 110.49 0))
-    (property "Footprint" "" (id 2) (at 177.8 105.41 0)
-      (effects (font (size 1.27 1.27)) hide)
-    )
-    (property "Datasheet" "" (id 3) (at 177.8 105.41 0)
-      (effects (font (size 1.27 1.27)) hide)
-    )
+  (symbol (lib_id "upsat-comms-hardware:GND") (at 142.24 113.03 0) (unit 1)
+    (in_bom yes) (on_board yes) (fields_autoplaced)
+    (property "Reference" "#PWR0170" (id 0) (at 142.24 119.38 0)
+      (effects (font (size 1.27 1.27)) hide)
+    )
+    (property "Value" "GND" (id 1) (at 142.24 117.475 0))
+    (property "Footprint" "" (id 2) (at 142.24 113.03 0))
+    (property "Datasheet" "" (id 3) (at 142.24 113.03 0))
     (pin "1")
   )
@@
     (pin "2")
   )
-  (symbol (lib_id "power:GND") (at 142.24 113.03 0) (unit 1)
-    (in_bom yes) (on_board yes) (fields_autoplaced)
-    (property "Reference" "#PWR0169" (id 0) (at 142.24 119.38 0)
-      (effects (font (size 1.27 1.27)) hide)
-    )
-    (property "Value" "GND" (id 1) (at 142.24 118.11 0))
-    (property "Footprint" "" (id 2) (at 142.24 113.03 0)
-      (effects (font (size 1.27 1.27)) hide)
-    )
-    (property "Datasheet" "" (id 3) (at 142.24 113.03 0)
-      (effects (font (size 1.27 1.27)) hide)
-    )
-    (pin "1")
-  )
-  (symbol (lib_id "power:GND") (at 194.31 97.79 0) (unit 1)
-    (in_bom yes) (on_board yes) (fields_autoplaced)
-    (property "Reference" "#PWR0171" (id 0) (at 194.31 104.14 0)
-      (effects (font (size 1.27 1.27)) hide)
-    )
-    (property "Value" "GND" (id 1) (at 194.31 102.87 0))
-    (property "Footprint" "" (id 2) (at 194.31 97.79 0)
-      (effects (font (size 1.27 1.27)) hide)
-    )
-    (property "Datasheet" "" (id 3) (at 194.31 97.79 0)
-      (effects (font (size 1.27 1.27)) hide)
-    )
-    (pin "1")
-  )
-  (symbol (lib_id "power:GND") (at 127 100.33 0) (unit 1)
-    (in_bom yes) (on_board yes) (fields_autoplaced)
-    (property "Reference" "#PWR0167" (id 0) (at 127 106.68 0)
-      (effects (font (size 1.27 1.27)) hide)
-    )
-    (property "Value" "GND" (id 1) (at 127 105.41 0))
-    (property "Footprint" "" (id 2) (at 127 100.33 0)
-      (effects (font (size 1.27 1.27)) hide)
-    )
-    (property "Datasheet" "" (id 3) (at 127 100.33 0)
-      (effects (font (size 1.27 1.27)) hide)
-    )
-    (pin "1")
-  )
-  (symbol (lib_id "power:GND") (at 212.09 135.89 0) (unit 1)
-    (in_bom yes) (on_board yes) (fields_autoplaced)
-    (property "Reference" "#PWR0172" (id 0) (at 212.09 142.24 0)
-      (effects (font (size 1.27 1.27)) hide)
-    )
-    (property "Value" "GND" (id 1) (at 212.09 140.97 0))
-    (property "Footprint" "" (id 2) (at 212.09 135.89 0)
-      (effects (font (size 1.27 1.27)) hide)
-    )
-    (property "Datasheet" "" (id 3) (at 212.09 135.89 0)
-      (effects (font (size 1.27 1.27)) hide)
-    )
-    (pin "1")
-  )
   (symbol (lib_id "Device:R") (at 212.09 128.27 180) (unit 1)

Commit message: Updated the changes
Parts:
- gave numbers to parts that had none: 2
- renumbered CB3 to CB1, CB1 to CB2, CB2 to CB3
Changed lines of the file:
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@@
   (symbol (lib_id "pspice:C") (at 115.57 135.89 0) (unit 1)
     (in_bom yes) (on_board yes) (fields_autoplaced)
-    (property "Reference" "CA?" (id 0) (at 120.65 134.6199 0)
+    (property "Reference" "CA5" (id 0) (at 120.65 134.6199 0)
       (effects (font (size 1.27 1.27)) (justify left))
     )
@@
   (symbol (lib_id "upsat-comms-hardware:GND") (at 177.8 105.41 0) (unit 1)
     (in_bom yes) (on_board yes) (fields_autoplaced)
-    (property "Reference" "#PWR0167" (id 0) (at 177.8 111.76 0)
+    (property "Reference" "#PWR072" (id 0) (at 177.8 111.76 0)
       (effects (font (size 1.27 1.27)) hide)
     )
@@
   (symbol (lib_id "upsat-comms-hardware:GND") (at 194.31 97.79 0) (unit 1)
     (in_bom yes) (on_board yes) (fields_autoplaced)
-    (property "Reference" "#PWR0171" (id 0) (at 194.31 104.14 0)
+    (property "Reference" "#PWR070" (id 0) (at 194.31 104.14 0)
       (effects (font (size 1.27 1.27)) hide)
     )
@@
   (symbol (lib_id "upsat-comms-hardware:GND") (at 143.51 142.875 0) (unit 1)
     (in_bom yes) (on_board yes) (fields_autoplaced)
-    (property "Reference" "#PWR0169" (id 0) (at 143.51 149.225 0)
+    (property "Reference" "#PWR075" (id 0) (at 143.51 149.225 0)
       (effects (font (size 1.27 1.27)) hide)
     )
@@
   (symbol (lib_id "upsat-comms-hardware:GND") (at 127 100.33 0) (unit 1)
     (in_bom yes) (on_board yes) (fields_autoplaced)
-    (property "Reference" "#PWR0168" (id 0) (at 127 106.68 0)
+    (property "Reference" "#PWR071" (id 0) (at 127 106.68 0)
       (effects (font (size 1.27 1.27)) hide)
     )
@@
   (symbol (lib_id "upsat-comms-hardware:GND") (at 212.09 135.89 0) (unit 1)
     (in_bom yes) (on_board yes) (fields_autoplaced)
-    (property "Reference" "#PWR0172" (id 0) (at 212.09 142.24 0)
+    (property "Reference" "#PWR074" (id 0) (at 212.09 142.24 0)
       (effects (font (size 1.27 1.27)) hide)
     )
@@
   (symbol (lib_id "pspice:C") (at 128.27 135.89 0) (unit 1)
     (in_bom yes) (on_board yes) (fields_autoplaced)
-    (property "Reference" "CB1" (id 0) (at 133.35 134.6199 0)
+    (property "Reference" "CB2" (id 0) (at 133.35 134.6199 0)
       (effects (font (size 1.27 1.27)) (justify left))
     )
@@
   (symbol (lib_id "DRV10970PWPR:DRV10970PWPR") (at 127 72.39 0) (unit 1)
     (in_bom yes) (on_board yes) (fields_autoplaced)
-    (property "Reference" "UA?" (id 0) (at 142.24 59.69 0))
+    (property "Reference" "UA2" (id 0) (at 142.24 59.69 0))
     (property "Value" "DRV10970PWPR" (id 1) (at 142.24 62.23 0))
     (property "Footprint" "DRV10970PWPR:SOP65P640X120-25N" (id 2) (at 127 72.39 0)
@@
   (symbol (lib_id "upsat-comms-hardware:GND") (at 142.24 113.03 0) (unit 1)
     (in_bom yes) (on_board yes) (fields_autoplaced)
-    (property "Reference" "#PWR0170" (id 0) (at 142.24 119.38 0)
+    (property "Reference" "#PWR073" (id 0) (at 142.24 119.38 0)
       (effects (font (size 1.27 1.27)) hide)
     )
@@
   (symbol (lib_id "pspice:C") (at 177.8 99.06 0) (unit 1)
     (in_bom yes) (on_board yes) (fields_autoplaced)
-    (property "Reference" "CB3" (id 0) (at 182.88 97.7899 0)
+    (property "Reference" "CB1" (id 0) (at 182.88 97.7899 0)
       (effects (font (size 1.27 1.27)) (justify left))
     )
@@
   (symbol (lib_id "pspice:C") (at 143.51 135.89 0) (unit 1)
     (in_bom yes) (on_board yes) (fields_autoplaced)
-    (property "Reference" "CB2" (id 0) (at 148.59 134.6199 0)
-      (effects (font (size 1.27 1.27)) (justify left))
-    )
+    (property "Reference" "CB3" (id 0) (at 148.59 134.6199 0)
+      (effects (font (size 1.27 1.27)) (justify left))
+    )

Commit message: Placed NCs at ADCS_HMC1051
Parts:
- renumbered CA5 to CB2, CB2 to CB3, CB3 to CB4, UA2 to UB1
Changed lines of the file:
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@@
   (symbol (lib_id "pspice:C") (at 115.57 135.89 0) (unit 1)
     (in_bom yes) (on_board yes) (fields_autoplaced)
-    (property "Reference" "CA5" (id 0) (at 120.65 134.6199 0)
+    (property "Reference" "CB2" (id 0) (at 120.65 134.6199 0)
       (effects (font (size 1.27 1.27)) (justify left))
     )
@@
   (symbol (lib_id "pspice:C") (at 128.27 135.89 0) (unit 1)
     (in_bom yes) (on_board yes) (fields_autoplaced)
-    (property "Reference" "CB2" (id 0) (at 133.35 134.6199 0)
+    (property "Reference" "CB3" (id 0) (at 133.35 134.6199 0)
       (effects (font (size 1.27 1.27)) (justify left))
     )
@@
   (symbol (lib_id "DRV10970PWPR:DRV10970PWPR") (at 127 72.39 0) (unit 1)
     (in_bom yes) (on_board yes) (fields_autoplaced)
-    (property "Reference" "UA2" (id 0) (at 142.24 59.69 0))
+    (property "Reference" "UB1" (id 0) (at 142.24 59.69 0))
     (property "Value" "DRV10970PWPR" (id 1) (at 142.24 62.23 0))
     (property "Footprint" "DRV10970PWPR:SOP65P640X120-25N" (id 2) (at 127 72.39 0)
@@
   (symbol (lib_id "pspice:C") (at 143.51 135.89 0) (unit 1)
     (in_bom yes) (on_board yes) (fields_autoplaced)
-    (property "Reference" "CB3" (id 0) (at 148.59 134.6199 0)
-      (effects (font (size 1.27 1.27)) (justify left))
-    )
+    (property "Reference" "CB4" (id 0) (at 148.59 134.6199 0)
+      (effects (font (size 1.27 1.27)) (justify left))
+    )
