File: DRV2.kicad_sch (KiCad schematic)
At the start: 15 parts

Commit message: Final Schematic
Other:
- note added: "A low-ESR ceramic capacitor must be placed in between the VM and VCP pins. TI recommends a value of 1-µF rated for 16 V. Place this component as close as possible to the pins."
Changed lines of the file:
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@@
     (stroke (width 0) (type default) (color 0 0 0 0))
+  )
+  (text "A low-ESR ceramic capacitor must be placed in between the VM and VCP pins. TI recommends a value of 1-µF\nrated for 16 V. Place this component as close as possible to the pins."
+    (at 85.09 46.355 0)
+    (effects (font (size 1.27 1.27) (thickness 0.254) bold italic) (justify left bottom))
   )
   (label "VINT" (at 194.31 81.28 0)

Commit message: MCU circuitry forgot LOL
Parts:
- renumbered CB4 to CB1, CB1 to CB2, CB2 to CB3, CB3 to CB4
Changed lines of the file:
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@@
   (symbol (lib_id "pspice:C") (at 115.57 135.89 0) (unit 1)
     (in_bom yes) (on_board yes) (fields_autoplaced)
-    (property "Reference" "CB1" (id 0) (at 120.65 134.6199 0)
+    (property "Reference" "CB2" (id 0) (at 120.65 134.6199 0)
       (effects (font (size 1.27 1.27)) (justify left))
     )
@@
   (symbol (lib_id "upsat-comms-hardware:GND") (at 177.8 105.41 0) (unit 1)
     (in_bom yes) (on_board yes) (fields_autoplaced)
-    (property "Reference" "#PWR087" (id 0) (at 177.8 111.76 0)
+    (property "Reference" "#PWR093" (id 0) (at 177.8 111.76 0)
       (effects (font (size 1.27 1.27)) hide)
     )
@@
   (symbol (lib_id "upsat-comms-hardware:GND") (at 194.31 97.79 0) (unit 1)
     (in_bom yes) (on_board yes) (fields_autoplaced)
-    (property "Reference" "#PWR088" (id 0) (at 194.31 104.14 0)
+    (property "Reference" "#PWR091" (id 0) (at 194.31 104.14 0)
       (effects (font (size 1.27 1.27)) hide)
     )
@@
   (symbol (lib_id "upsat-comms-hardware:GND") (at 143.51 142.875 0) (unit 1)
     (in_bom yes) (on_board yes) (fields_autoplaced)
-    (property "Reference" "#PWR086" (id 0) (at 143.51 149.225 0)
+    (property "Reference" "#PWR096" (id 0) (at 143.51 149.225 0)
       (effects (font (size 1.27 1.27)) hide)
     )
@@
   (symbol (lib_id "upsat-comms-hardware:GND") (at 127 100.33 0) (unit 1)
     (in_bom yes) (on_board yes) (fields_autoplaced)
-    (property "Reference" "#PWR084" (id 0) (at 127 106.68 0)
+    (property "Reference" "#PWR092" (id 0) (at 127 106.68 0)
       (effects (font (size 1.27 1.27)) hide)
     )
@@
   (symbol (lib_id "upsat-comms-hardware:GND") (at 212.09 135.89 0) (unit 1)
     (in_bom yes) (on_board yes) (fields_autoplaced)
-    (property "Reference" "#PWR089" (id 0) (at 212.09 142.24 0)
+    (property "Reference" "#PWR095" (id 0) (at 212.09 142.24 0)
       (effects (font (size 1.27 1.27)) hide)
     )
@@
   (symbol (lib_id "pspice:C") (at 128.27 135.89 0) (unit 1)
     (in_bom yes) (on_board yes) (fields_autoplaced)
-    (property "Reference" "CB2" (id 0) (at 133.35 134.6199 0)
+    (property "Reference" "CB3" (id 0) (at 133.35 134.6199 0)
       (effects (font (size 1.27 1.27)) (justify left))
     )
@@
   (symbol (lib_id "upsat-comms-hardware:GND") (at 142.24 113.03 0) (unit 1)
     (in_bom yes) (on_board yes) (fields_autoplaced)
-    (property "Reference" "#PWR085" (id 0) (at 142.24 119.38 0)
+    (property "Reference" "#PWR094" (id 0) (at 142.24 119.38 0)
       (effects (font (size 1.27 1.27)) hide)
     )
@@
   (symbol (lib_id "pspice:C") (at 177.8 99.06 0) (unit 1)
     (in_bom yes) (on_board yes) (fields_autoplaced)
-    (property "Reference" "CB4" (id 0) (at 182.88 97.7899 0)
+    (property "Reference" "CB1" (id 0) (at 182.88 97.7899 0)
       (effects (font (size 1.27 1.27)) (justify left))
     )
@@
   (symbol (lib_id "pspice:C") (at 143.51 135.89 0) (unit 1)
     (in_bom yes) (on_board yes) (fields_autoplaced)
-    (property "Reference" "CB3" (id 0) (at 148.59 134.6199 0)
-      (effects (font (size 1.27 1.27)) (justify left))
-    )
+    (property "Reference" "CB4" (id 0) (at 148.59 134.6199 0)
+      (effects (font (size 1.27 1.27)) (justify left))
+    )

Commit message: All frequency sensitive caps and specific inductor PNs added
Other:
- note added: "0603B105K160XD"
Changed lines of the file:
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@@
     (effects (font (size 1.27 1.27) (thickness 0.254) bold italic) (justify left bottom))
+  )
+  (text "0603B105K160XD" (at 102.87 135.89 0)
+    (effects (font (size 1.27 1.27)) (justify left bottom))
   )
   (label "VINT" (at 194.31 81.28 0)
