File: Motor_connectors.kicad_sch (KiCad schematic)
At the start: 3 parts

Commit message: MCU circuitry forgot LOL
Parts:
- renumbered JR3 to JR2, JR2 to JR3
Changed lines of the file:
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@@
   (symbol (lib_id "upsat-comms-hardware:GND") (at 126.365 84.074 0) (unit 1)
     (in_bom yes) (on_board yes) (fields_autoplaced)
-    (property "Reference" "#PWR0115" (id 0) (at 126.365 90.424 0)
+    (property "Reference" "#PWR0119" (id 0) (at 126.365 90.424 0)
       (effects (font (size 1.27 1.27)) hide)
     )
@@
   (symbol (lib_id "upsat-comms-hardware:GND") (at 86.995 86.614 0) (unit 1)
     (in_bom yes) (on_board yes) (fields_autoplaced)
-    (property "Reference" "#PWR0113" (id 0) (at 86.995 92.964 0)
+    (property "Reference" "#PWR0121" (id 0) (at 86.995 92.964 0)
       (effects (font (size 1.27 1.27)) hide)
     )
@@
   (symbol (lib_id "upsat-comms-hardware:GND") (at 174.625 86.614 0) (unit 1)
     (in_bom yes) (on_board yes) (fields_autoplaced)
-    (property "Reference" "#PWR0116" (id 0) (at 174.625 92.964 0)
+    (property "Reference" "#PWR0122" (id 0) (at 174.625 92.964 0)
       (effects (font (size 1.27 1.27)) hide)
     )
@@
   (symbol (lib_id "upsat-comms-hardware:GND") (at 37.465 82.804 0) (unit 1)
     (in_bom yes) (on_board yes) (fields_autoplaced)
-    (property "Reference" "#PWR0111" (id 0) (at 37.465 89.154 0)
+    (property "Reference" "#PWR0118" (id 0) (at 37.465 89.154 0)
       (effects (font (size 1.27 1.27)) hide)
     )
@@
   (symbol (lib_id "2367196-8:2367196-8") (at 228.6 78.994 0) (unit 1)
     (in_bom yes) (on_board yes) (fields_autoplaced)
-    (property "Reference" "JR2" (id 0) (at 240.03 66.294 0))
+    (property "Reference" "JR3" (id 0) (at 240.03 66.294 0))
     (property "Value" "2367196-8" (id 1) (at 240.03 68.834 0))
     (property "Footprint" "2367196-8:23671968" (id 2) (at 228.6 78.994 0)
@@
   (symbol (lib_id "upsat-comms-hardware:GND") (at 271.78 86.614 0) (unit 1)
     (in_bom yes) (on_board yes) (fields_autoplaced)
-    (property "Reference" "#PWR0114" (id 0) (at 271.78 92.964 0)
+    (property "Reference" "#PWR0123" (id 0) (at 271.78 92.964 0)
       (effects (font (size 1.27 1.27)) hide)
     )
@@
   (symbol (lib_id "2367196-8:2367196-8") (at 135.255 78.994 0) (unit 1)
     (in_bom yes) (on_board yes) (fields_autoplaced)
-    (property "Reference" "JR3" (id 0) (at 146.685 66.294 0))
+    (property "Reference" "JR2" (id 0) (at 146.685 66.294 0))
     (property "Value" "2367196-8" (id 1) (at 146.685 68.834 0))
     (property "Footprint" "2367196-8:23671968" (id 2) (at 135.255 78.994 0)
@@
   (symbol (lib_id "upsat-comms-hardware:GND") (at 223.52 84.074 0) (unit 1)
     (in_bom yes) (on_board yes) (fields_autoplaced)
-    (property "Reference" "#PWR0112" (id 0) (at 223.52 90.424 0)
+    (property "Reference" "#PWR0120" (id 0) (at 223.52 90.424 0)
       (effects (font (size 1.27 1.27)) hide)
     )
