File: SS_Connector.kicad_sch (KiCad schematic)
At the start: 6 parts

Commit message: ERC cleared in magnetometer connectors sheet
Parts:
- renumbered JSC2 to JSC1, JSC3 to JSC2, JSC4 to JSC3, JSC5 to JSC4, JSC6 to JSC5, JSC7 to JSC6
Changed lines of the file:
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@@
   (symbol (lib_id "2367196-8:2367196-8") (at 207.01 114.3 0) (unit 1)
     (in_bom yes) (on_board yes) (fields_autoplaced)
-    (property "Reference" "JSC6" (id 0) (at 218.44 101.6 0))
+    (property "Reference" "JSC5" (id 0) (at 218.44 101.6 0))
     (property "Value" "2367196-8" (id 1) (at 218.44 104.14 0))
     (property "Footprint" "" (id 2) (at 207.01 114.3 0)
@@
   (symbol (lib_id "2367196-8:2367196-8") (at 115.57 43.18 0) (unit 1)
     (in_bom yes) (on_board yes) (fields_autoplaced)
-    (property "Reference" "JSC3" (id 0) (at 127 30.48 0))
+    (property "Reference" "JSC2" (id 0) (at 127 30.48 0))
     (property "Value" "2367196-8" (id 1) (at 127 33.02 0))
     (property "Footprint" "" (id 2) (at 115.57 43.18 0)
@@
   (symbol (lib_id "upsat-comms-hardware:GND") (at 110.49 46.99 0) (unit 1)
     (in_bom yes) (on_board yes) (fields_autoplaced)
-    (property "Reference" "#PWR0155" (id 0) (at 110.49 53.34 0)
+    (property "Reference" "#PWR0157" (id 0) (at 110.49 53.34 0)
       (effects (font (size 1.27 1.27)) hide)
     )
@@
   (symbol (lib_id "upsat-comms-hardware:GND") (at 199.39 48.26 0) (unit 1)
     (in_bom yes) (on_board yes) (fields_autoplaced)
-    (property "Reference" "#PWR0157" (id 0) (at 199.39 54.61 0)
+    (property "Reference" "#PWR0159" (id 0) (at 199.39 54.61 0)
       (effects (font (size 1.27 1.27)) hide)
     )
@@
   (symbol (lib_id "upsat-comms-hardware:GND") (at 73.66 136.525 0) (unit 1)
     (in_bom yes) (on_board yes) (fields_autoplaced)
-    (property "Reference" "#PWR0166" (id 0) (at 73.66 142.875 0)
+    (property "Reference" "#PWR0168" (id 0) (at 73.66 142.875 0)
       (effects (font (size 1.27 1.27)) hide)
     )
@@
   (symbol (lib_id "upsat-comms-hardware:GND") (at 78.74 63.5 0) (unit 1)
     (in_bom yes) (on_board yes) (fields_autoplaced)
-    (property "Reference" "#PWR0158" (id 0) (at 78.74 69.85 0)
+    (property "Reference" "#PWR0160" (id 0) (at 78.74 69.85 0)
       (effects (font (size 1.27 1.27)) hide)
     )
@@
   (symbol (lib_id "upsat-comms-hardware:GND") (at 41.91 121.92 0) (unit 1)
     (in_bom yes) (on_board yes) (fields_autoplaced)
-    (property "Reference" "#PWR0163" (id 0) (at 41.91 128.27 0)
+    (property "Reference" "#PWR0165" (id 0) (at 41.91 128.27 0)
       (effects (font (size 1.27 1.27)) hide)
     )
@@
   (symbol (lib_id "upsat-comms-hardware:GND") (at 114.3 119.38 0) (unit 1)
     (in_bom yes) (on_board yes) (fields_autoplaced)
-    (property "Reference" "#PWR0161" (id 0) (at 114.3 125.73 0)
+    (property "Reference" "#PWR0163" (id 0) (at 114.3 125.73 0)
       (effects (font (size 1.27 1.27)) hide)
     )
@@
   (symbol (lib_id "2367196-8:2367196-8") (at 118.11 114.3 0) (unit 1)
     (in_bom yes) (on_board yes) (fields_autoplaced)
-    (property "Reference" "JSC5" (id 0) (at 129.54 101.6 0))
+    (property "Reference" "JSC4" (id 0) (at 129.54 101.6 0))
     (property "Value" "2367196-8" (id 1) (at 129.54 104.14 0))
     (property "Footprint" "" (id 2) (at 118.11 114.3 0)
@@
   (symbol (lib_id "2367196-8:2367196-8") (at 201.93 43.18 0) (unit 1)
     (in_bom yes) (on_board yes) (fields_autoplaced)
-    (property "Reference" "JSC4" (id 0) (at 213.36 30.48 0))
+    (property "Reference" "JSC3" (id 0) (at 213.36 30.48 0))
     (property "Value" "2367196-8" (id 1) (at 213.36 33.02 0))
     (property "Footprint" "" (id 2) (at 201.93 43.18 0)
@@
   (symbol (lib_id "2367196-8:2367196-8") (at 53.34 43.18 0) (unit 1)
     (in_bom yes) (on_board yes) (fields_autoplaced)
-    (property "Reference" "JSC2" (id 0) (at 64.77 30.48 0))
+    (property "Reference" "JSC1" (id 0) (at 64.77 30.48 0))
     (property "Value" "2367196-8" (id 1) (at 64.77 33.02 0))
     (property "Footprint" "" (id 2) (at 53.34 43.18 0)
@@
   (symbol (lib_id "upsat-comms-hardware:GND") (at 50.8 48.26 0) (unit 1)
     (in_bom yes) (on_board yes) (fields_autoplaced)
-    (property "Reference" "#PWR0156" (id 0) (at 50.8 54.61 0)
+    (property "Reference" "#PWR0158" (id 0) (at 50.8 54.61 0)
       (effects (font (size 1.27 1.27)) hide)
     )
@@
   (symbol (lib_id "upsat-comms-hardware:GND") (at 142.24 63.5 0) (unit 1)
     (in_bom yes) (on_board yes) (fields_autoplaced)
-    (property "Reference" "#PWR0159" (id 0) (at 142.24 69.85 0)
+    (property "Reference" "#PWR0161" (id 0) (at 142.24 69.85 0)
       (effects (font (size 1.27 1.27)) hide)
     )
@@
   (symbol (lib_id "upsat-comms-hardware:GND") (at 232.41 133.35 0) (unit 1)
     (in_bom yes) (on_board yes) (fields_autoplaced)
-    (property "Reference" "#PWR0164" (id 0) (at 232.41 139.7 0)
+    (property "Reference" "#PWR0166" (id 0) (at 232.41 139.7 0)
       (effects (font (size 1.27 1.27)) hide)
     )
@@
   (symbol (lib_id "upsat-comms-hardware:GND") (at 229.87 63.5 0) (unit 1)
     (in_bom yes) (on_board yes) (fields_autoplaced)
-    (property "Reference" "#PWR0160" (id 0) (at 229.87 69.85 0)
+    (property "Reference" "#PWR0162" (id 0) (at 229.87 69.85 0)
       (effects (font (size 1.27 1.27)) hide)
     )
@@
   (symbol (lib_id "2367196-8:2367196-8") (at 46.99 116.84 0) (unit 1)
     (in_bom yes) (on_board yes) (fields_autoplaced)
-    (property "Reference" "JSC7" (id 0) (at 58.42 104.14 0))
+    (property "Reference" "JSC6" (id 0) (at 58.42 104.14 0))
     (property "Value" "2367196-8" (id 1) (at 58.42 106.68 0))
     (property "Footprint" "" (id 2) (at 46.99 116.84 0)
@@
   (symbol (lib_id "upsat-comms-hardware:GND") (at 144.78 135.89 0) (unit 1)
     (in_bom yes) (on_board yes) (fields_autoplaced)
-    (property "Reference" "#PWR0165" (id 0) (at 144.78 142.24 0)
+    (property "Reference" "#PWR0167" (id 0) (at 144.78 142.24 0)
       (effects (font (size 1.27 1.27)) hide)
     )
@@
   (symbol (lib_id "upsat-comms-hardware:GND") (at 204.47 119.38 0) (unit 1)
     (in_bom yes) (on_board yes) (fields_autoplaced)
-    (property "Reference" "#PWR0162" (id 0) (at 204.47 125.73 0)
-      (effects (font (size 1.27 1.27)) hide)
-    )
+    (property "Reference" "#PWR0164" (id 0) (at 204.47 125.73 0)
+      (effects (font (size 1.27 1.27)) hide)
+    )

Commit message: Page settings changed. Added some testpoints. Some comments are made.
Parts:
- renumbered JSC6 to JSC1, JSC1 to JSC2, JSC2 to JSC3, JSC3 to JSC5, JSC5 to JSC6
Changed lines of the file:
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@@
   (symbol (lib_id "2367196-8:2367196-8") (at 207.01 114.3 0) (unit 1)
     (in_bom yes) (on_board yes) (fields_autoplaced)
-    (property "Reference" "JSC5" (id 0) (at 218.44 101.6 0))
+    (property "Reference" "JSC6" (id 0) (at 218.44 101.6 0))
     (property "Value" "2367196-8" (id 1) (at 218.44 104.14 0))
     (property "Footprint" "" (id 2) (at 207.01 114.3 0)
@@
   (symbol (lib_id "2367196-8:2367196-8") (at 115.57 43.18 0) (unit 1)
     (in_bom yes) (on_board yes) (fields_autoplaced)
-    (property "Reference" "JSC2" (id 0) (at 127 30.48 0))
+    (property "Reference" "JSC3" (id 0) (at 127 30.48 0))
     (property "Value" "2367196-8" (id 1) (at 127 33.02 0))
     (property "Footprint" "" (id 2) (at 115.57 43.18 0)
@@
   (symbol (lib_id "upsat-comms-hardware:GND") (at 110.49 46.99 0) (unit 1)
     (in_bom yes) (on_board yes) (fields_autoplaced)
-    (property "Reference" "#PWR0157" (id 0) (at 110.49 53.34 0)
+    (property "Reference" "#PWR0174" (id 0) (at 110.49 53.34 0)
       (effects (font (size 1.27 1.27)) hide)
     )
@@
   (symbol (lib_id "upsat-comms-hardware:GND") (at 199.39 48.26 0) (unit 1)
     (in_bom yes) (on_board yes) (fields_autoplaced)
-    (property "Reference" "#PWR0159" (id 0) (at 199.39 54.61 0)
+    (property "Reference" "#PWR0178" (id 0) (at 199.39 54.61 0)
       (effects (font (size 1.27 1.27)) hide)
     )
@@
   (symbol (lib_id "upsat-comms-hardware:GND") (at 73.66 136.525 0) (unit 1)
     (in_bom yes) (on_board yes) (fields_autoplaced)
-    (property "Reference" "#PWR0168" (id 0) (at 73.66 142.875 0)
+    (property "Reference" "#PWR0172" (id 0) (at 73.66 142.875 0)
       (effects (font (size 1.27 1.27)) hide)
     )
@@
   (symbol (lib_id "upsat-comms-hardware:GND") (at 78.74 63.5 0) (unit 1)
     (in_bom yes) (on_board yes) (fields_autoplaced)
-    (property "Reference" "#PWR0160" (id 0) (at 78.74 69.85 0)
+    (property "Reference" "#PWR0173" (id 0) (at 78.74 69.85 0)
       (effects (font (size 1.27 1.27)) hide)
     )
@@
   (symbol (lib_id "upsat-comms-hardware:GND") (at 41.91 121.92 0) (unit 1)
     (in_bom yes) (on_board yes) (fields_autoplaced)
-    (property "Reference" "#PWR0165" (id 0) (at 41.91 128.27 0)
+    (property "Reference" "#PWR0170" (id 0) (at 41.91 128.27 0)
       (effects (font (size 1.27 1.27)) hide)
     )
@@
   (symbol (lib_id "upsat-comms-hardware:GND") (at 114.3 119.38 0) (unit 1)
     (in_bom yes) (on_board yes) (fields_autoplaced)
-    (property "Reference" "#PWR0163" (id 0) (at 114.3 125.73 0)
+    (property "Reference" "#PWR0175" (id 0) (at 114.3 125.73 0)
       (effects (font (size 1.27 1.27)) hide)
     )
@@
   (symbol (lib_id "2367196-8:2367196-8") (at 201.93 43.18 0) (unit 1)
     (in_bom yes) (on_board yes) (fields_autoplaced)
-    (property "Reference" "JSC3" (id 0) (at 213.36 30.48 0))
+    (property "Reference" "JSC5" (id 0) (at 213.36 30.48 0))
     (property "Value" "2367196-8" (id 1) (at 213.36 33.02 0))
     (property "Footprint" "" (id 2) (at 201.93 43.18 0)
@@
   (symbol (lib_id "2367196-8:2367196-8") (at 53.34 43.18 0) (unit 1)
     (in_bom yes) (on_board yes) (fields_autoplaced)
-    (property "Reference" "JSC1" (id 0) (at 64.77 30.48 0))
+    (property "Reference" "JSC2" (id 0) (at 64.77 30.48 0))
     (property "Value" "2367196-8" (id 1) (at 64.77 33.02 0))
     (property "Footprint" "" (id 2) (at 53.34 43.18 0)
@@
   (symbol (lib_id "upsat-comms-hardware:GND") (at 50.8 48.26 0) (unit 1)
     (in_bom yes) (on_board yes) (fields_autoplaced)
-    (property "Reference" "#PWR0158" (id 0) (at 50.8 54.61 0)
+    (property "Reference" "#PWR0171" (id 0) (at 50.8 54.61 0)
       (effects (font (size 1.27 1.27)) hide)
     )
@@
   (symbol (lib_id "upsat-comms-hardware:GND") (at 142.24 63.5 0) (unit 1)
     (in_bom yes) (on_board yes) (fields_autoplaced)
-    (property "Reference" "#PWR0161" (id 0) (at 142.24 69.85 0)
+    (property "Reference" "#PWR0176" (id 0) (at 142.24 69.85 0)
       (effects (font (size 1.27 1.27)) hide)
     )
@@
   (symbol (lib_id "upsat-comms-hardware:GND") (at 232.41 133.35 0) (unit 1)
     (in_bom yes) (on_board yes) (fields_autoplaced)
-    (property "Reference" "#PWR0166" (id 0) (at 232.41 139.7 0)
+    (property "Reference" "#PWR0181" (id 0) (at 232.41 139.7 0)
       (effects (font (size 1.27 1.27)) hide)
     )
@@
   (symbol (lib_id "upsat-comms-hardware:GND") (at 229.87 63.5 0) (unit 1)
     (in_bom yes) (on_board yes) (fields_autoplaced)
-    (property "Reference" "#PWR0162" (id 0) (at 229.87 69.85 0)
+    (property "Reference" "#PWR0180" (id 0) (at 229.87 69.85 0)
       (effects (font (size 1.27 1.27)) hide)
     )
@@
   (symbol (lib_id "2367196-8:2367196-8") (at 46.99 116.84 0) (unit 1)
     (in_bom yes) (on_board yes) (fields_autoplaced)
-    (property "Reference" "JSC6" (id 0) (at 58.42 104.14 0))
+    (property "Reference" "JSC1" (id 0) (at 58.42 104.14 0))
     (property "Value" "2367196-8" (id 1) (at 58.42 106.68 0))
     (property "Footprint" "" (id 2) (at 46.99 116.84 0)
@@
   (symbol (lib_id "upsat-comms-hardware:GND") (at 144.78 135.89 0) (unit 1)
     (in_bom yes) (on_board yes) (fields_autoplaced)
-    (property "Reference" "#PWR0167" (id 0) (at 144.78 142.24 0)
+    (property "Reference" "#PWR0177" (id 0) (at 144.78 142.24 0)
       (effects (font (size 1.27 1.27)) hide)
     )
@@
   (symbol (lib_id "upsat-comms-hardware:GND") (at 204.47 119.38 0) (unit 1)
     (in_bom yes) (on_board yes) (fields_autoplaced)
-    (property "Reference" "#PWR0164" (id 0) (at 204.47 125.73 0)
-      (effects (font (size 1.27 1.27)) hide)
-    )
+    (property "Reference" "#PWR0179" (id 0) (at 204.47 125.73 0)
+      (effects (font (size 1.27 1.27)) hide)
+    )

Commit message: I2C lines are pulled up
Parts:
- JSC1, JSC2, JSC3, JSC4, JSC5, JSC6: footprint (none) -> 2367196-8:23671968
Changed lines of the file:
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@@
     (property "Reference" "JSC6" (id 0) (at 218.44 101.6 0))
     (property "Value" "2367196-8" (id 1) (at 218.44 104.14 0))
-    (property "Footprint" "" (id 2) (at 207.01 114.3 0)
+    (property "Footprint" "2367196-8:23671968" (id 2) (at 207.01 114.3 0)
       (effects (font (size 1.27 1.27)) hide)
     )
@@
     (property "Reference" "JSC3" (id 0) (at 127 30.48 0))
     (property "Value" "2367196-8" (id 1) (at 127 33.02 0))
-    (property "Footprint" "" (id 2) (at 115.57 43.18 0)
+    (property "Footprint" "2367196-8:23671968" (id 2) (at 115.57 43.18 0)
       (effects (font (size 1.27 1.27)) hide)
     )
@@
   (symbol (lib_id "upsat-comms-hardware:GND") (at 110.49 46.99 0) (unit 1)
     (in_bom yes) (on_board yes) (fields_autoplaced)
-    (property "Reference" "#PWR0174" (id 0) (at 110.49 53.34 0)
+    (property "Reference" "#PWR0176" (id 0) (at 110.49 53.34 0)
       (effects (font (size 1.27 1.27)) hide)
     )
@@
   (symbol (lib_id "upsat-comms-hardware:GND") (at 199.39 48.26 0) (unit 1)
     (in_bom yes) (on_board yes) (fields_autoplaced)
-    (property "Reference" "#PWR0178" (id 0) (at 199.39 54.61 0)
+    (property "Reference" "#PWR0180" (id 0) (at 199.39 54.61 0)
       (effects (font (size 1.27 1.27)) hide)
     )
@@
   (symbol (lib_id "upsat-comms-hardware:GND") (at 73.66 136.525 0) (unit 1)
     (in_bom yes) (on_board yes) (fields_autoplaced)
-    (property "Reference" "#PWR0172" (id 0) (at 73.66 142.875 0)
+    (property "Reference" "#PWR0174" (id 0) (at 73.66 142.875 0)
       (effects (font (size 1.27 1.27)) hide)
     )
@@
   (symbol (lib_id "upsat-comms-hardware:GND") (at 78.74 63.5 0) (unit 1)
     (in_bom yes) (on_board yes) (fields_autoplaced)
-    (property "Reference" "#PWR0173" (id 0) (at 78.74 69.85 0)
+    (property "Reference" "#PWR0175" (id 0) (at 78.74 69.85 0)
       (effects (font (size 1.27 1.27)) hide)
     )
@@
   (symbol (lib_id "upsat-comms-hardware:GND") (at 41.91 121.92 0) (unit 1)
     (in_bom yes) (on_board yes) (fields_autoplaced)
-    (property "Reference" "#PWR0170" (id 0) (at 41.91 128.27 0)
+    (property "Reference" "#PWR0172" (id 0) (at 41.91 128.27 0)
       (effects (font (size 1.27 1.27)) hide)
     )
@@
   (symbol (lib_id "upsat-comms-hardware:GND") (at 114.3 119.38 0) (unit 1)
     (in_bom yes) (on_board yes) (fields_autoplaced)
-    (property "Reference" "#PWR0175" (id 0) (at 114.3 125.73 0)
+    (property "Reference" "#PWR0177" (id 0) (at 114.3 125.73 0)
       (effects (font (size 1.27 1.27)) hide)
     )
@@
     (property "Reference" "JSC4" (id 0) (at 129.54 101.6 0))
     (property "Value" "2367196-8" (id 1) (at 129.54 104.14 0))
-    (property "Footprint" "" (id 2) (at 118.11 114.3 0)
+    (property "Footprint" "2367196-8:23671968" (id 2) (at 118.11 114.3 0)
       (effects (font (size 1.27 1.27)) hide)
     )
@@
     (property "Reference" "JSC5" (id 0) (at 213.36 30.48 0))
     (property "Value" "2367196-8" (id 1) (at 213.36 33.02 0))
-    (property "Footprint" "" (id 2) (at 201.93 43.18 0)
+    (property "Footprint" "2367196-8:23671968" (id 2) (at 201.93 43.18 0)
       (effects (font (size 1.27 1.27)) hide)
     )
@@
     (property "Reference" "JSC2" (id 0) (at 64.77 30.48 0))
     (property "Value" "2367196-8" (id 1) (at 64.77 33.02 0))
-    (property "Footprint" "" (id 2) (at 53.34 43.18 0)
+    (property "Footprint" "2367196-8:23671968" (id 2) (at 53.34 43.18 0)
       (effects (font (size 1.27 1.27)) hide)
     )
@@
   (symbol (lib_id "upsat-comms-hardware:GND") (at 50.8 48.26 0) (unit 1)
     (in_bom yes) (on_board yes) (fields_autoplaced)
-    (property "Reference" "#PWR0171" (id 0) (at 50.8 54.61 0)
+    (property "Reference" "#PWR0173" (id 0) (at 50.8 54.61 0)
       (effects (font (size 1.27 1.27)) hide)
     )
@@
   (symbol (lib_id "upsat-comms-hardware:GND") (at 142.24 63.5 0) (unit 1)
     (in_bom yes) (on_board yes) (fields_autoplaced)
-    (property "Reference" "#PWR0176" (id 0) (at 142.24 69.85 0)
+    (property "Reference" "#PWR0178" (id 0) (at 142.24 69.85 0)
       (effects (font (size 1.27 1.27)) hide)
     )
@@
   (symbol (lib_id "upsat-comms-hardware:GND") (at 232.41 133.35 0) (unit 1)
     (in_bom yes) (on_board yes) (fields_autoplaced)
-    (property "Reference" "#PWR0181" (id 0) (at 232.41 139.7 0)
+    (property "Reference" "#PWR0183" (id 0) (at 232.41 139.7 0)
       (effects (font (size 1.27 1.27)) hide)
     )
@@
   (symbol (lib_id "upsat-comms-hardware:GND") (at 229.87 63.5 0) (unit 1)
     (in_bom yes) (on_board yes) (fields_autoplaced)
-    (property "Reference" "#PWR0180" (id 0) (at 229.87 69.85 0)
+    (property "Reference" "#PWR0182" (id 0) (at 229.87 69.85 0)
       (effects (font (size 1.27 1.27)) hide)
     )
@@
     (property "Reference" "JSC1" (id 0) (at 58.42 104.14 0))
     (property "Value" "2367196-8" (id 1) (at 58.42 106.68 0))
-    (property "Footprint" "" (id 2) (at 46.99 116.84 0)
+    (property "Footprint" "2367196-8:23671968" (id 2) (at 46.99 116.84 0)
       (effects (font (size 1.27 1.27)) hide)
     )
@@
   (symbol (lib_id "upsat-comms-hardware:GND") (at 144.78 135.89 0) (unit 1)
     (in_bom yes) (on_board yes) (fields_autoplaced)
-    (property "Reference" "#PWR0177" (id 0) (at 144.78 142.24 0)
+    (property "Reference" "#PWR0179" (id 0) (at 144.78 142.24 0)
       (effects (font (size 1.27 1.27)) hide)
     )
@@
   (symbol (lib_id "upsat-comms-hardware:GND") (at 204.47 119.38 0) (unit 1)
     (in_bom yes) (on_board yes) (fields_autoplaced)
-    (property "Reference" "#PWR0179" (id 0) (at 204.47 125.73 0)
-      (effects (font (size 1.27 1.27)) hide)
-    )
+    (property "Reference" "#PWR0181" (id 0) (at 204.47 125.73 0)
+      (effects (font (size 1.27 1.27)) hide)
+    )
