File: Interboard.kicad_sch (KiCad schematic)
At the start: 2 parts

Commit message: Finalisations done, please produce BOM and fabricate
Connections:
- net GND: now also JIB1.2, JIB1.4; no longer JIB1.10, JIB1.9
- net at UIB1.2 (FILTER_2_1): now also JIB1.3; no longer JIB1.2
- net at UIB1.3 (FILTER_3_1): now also JIB1.5; no longer JIB1.3
- net at UIB1.4 (FILTER_4_1): now also JIB1.6; no longer JIB1.4
- net at UIB1.5 (FILTER_5_1): now also JIB1.7; no longer JIB1.5
- net at UIB1.6 (FILTER_6_1): now also JIB1.8; no longer JIB1.6
- net at UIB1.7 (FILTER_7_1): now also JIB1.9; no longer JIB1.7
- net at UIB1.8 (FILTER_8_1): now also JIB1.10; no longer JIB1.8
Other:
- note added: "Route ESD Diode close to connector"
- note added: "Sheet Comments :"
- note removed: "Chinmay : Check if theres a 4th line for SPI"
- moved on the sheet: JIB1, UIB1

Commit message: inductor part numbers added
Connections:
- net SPI2_CS: no longer names the net of UIB1.9 (FILTER_8_2)
- net SPI2_MISO: no longer names the net of UIB1.10 (FILTER_7_2)
- net SPI2_MOSI: no longer names the net of UIB1.11 (FILTER_6_2)
- net SPI2_SCK renamed ADCS_BOOT_MODE
- no-connect marks 0 -> 3
Changed lines of the file:
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@@
   (junction (at 153.67 81.28) (diameter 0) (color 0 0 0 0)
   )
+  (no_connect (at 209.55 86.36))
+  (no_connect (at 209.55 91.44))
+  (no_connect (at 209.55 88.9))
   (wire (pts (xy 207.01 81.28) (xy 209.55 81.28))
     (stroke (width 0) (type default) (color 0 0 0 0))
@@
     (effects (font (size 1.27 1.27)) (justify left))
   )
-  (hierarchical_label "SPI2_MOSI" (shape bidirectional) (at 209.55 86.36 0)
-    (effects (font (size 1.27 1.27)) (justify left))
-  )
-  (hierarchical_label "SPI2_SCK" (shape bidirectional) (at 209.55 83.82 0)
-    (effects (font (size 1.27 1.27)) (justify left))
-  )
   (hierarchical_label "I2C_SDA_3V3" (shape bidirectional) (at 209.55 81.28 0)
     (effects (font (size 1.27 1.27)) (justify left))
   )
-  (hierarchical_label "SPI2_CS" (shape bidirectional) (at 209.55 91.44 0)
+  (hierarchical_label "ADCS_BOOT_MODE" (shape bidirectional) (at 209.55 83.82 0)
     (effects (font (size 1.27 1.27)) (justify left))
   )
-  (hierarchical_label "SPI2_MISO" (shape bidirectional) (at 209.55 88.9 0)
-    (effects (font (size 1.27 1.27)) (justify left))
-  )
