File: Power.kicad_sch (KiCad schematic)
At the start: 25 parts

Commit message: I2C lines are pulled up
Parts:
- CP1, CP2, CP3, CP4, CP5, CP6, CP7, CP8, CP9: footprint (none) -> Capacitor_SMD:C_0603_1608Metric
- LP1, LP2, LP3: footprint (none) -> Inductor_SMD:L_0805_2012Metric_Pad1.15x1.40mm_HandSolder
- RP1, RP10, RP2, RP3, RP4, RP5, RP6, RP7, RP8, RP9: footprint (none) -> Resistor_SMD:R_0603_1608Metric

Commit message: Final Schematic
Other:
- note removed: "Check this Change once"
- moved on the sheet: RP5, RP6, RP7, RP8
Changed lines of the file:
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@@
   (junction (at 63.5 33.02) (diameter 0) (color 0 0 0 0)
   )
-  (junction (at 174.625 83.82) (diameter 0) (color 0 0 0 0)
+  (junction (at 224.663 143.637) (diameter 0) (color 0 0 0 0)
   )
   (junction (at 170.18 31.75) (diameter 0) (color 0 0 0 0)
@@
     (stroke (width 0) (type default) (color 0 0 0 0))
   )
-  (wire (pts (xy 191.135 89.535) (xy 196.85 89.535))
+  (wire (pts (xy 241.173 149.352) (xy 246.888 149.352))
     (stroke (width 0) (type default) (color 0 0 0 0))
   )
@@
     (stroke (width 0) (type default) (color 0 0 0 0))
   )
-  (wire (pts (xy 174.625 89.535) (xy 183.515 89.535))
+  (wire (pts (xy 224.663 149.352) (xy 233.553 149.352))
     (stroke (width 0) (type default) (color 0 0 0 0))
   )
@@
     (stroke (width 0) (type default) (color 0 0 0 0))
   )
-  (wire (pts (xy 158.75 83.82) (xy 165.1 83.82))
+  (wire (pts (xy 208.788 143.637) (xy 215.138 143.637))
     (stroke (width 0) (type default) (color 0 0 0 0))
   )
@@
     (stroke (width 0) (type default) (color 0 0 0 0))
   )
-  (wire (pts (xy 191.77 83.82) (xy 196.85 83.82))
+  (wire (pts (xy 241.808 143.637) (xy 246.888 143.637))
     (stroke (width 0) (type default) (color 0 0 0 0))
   )
@@
     (stroke (width 0) (type default) (color 0 0 0 0))
   )
-  (wire (pts (xy 174.625 73.025) (xy 174.625 83.82))
+  (wire (pts (xy 224.663 132.842) (xy 224.663 143.637))
     (stroke (width 0) (type default) (color 0 0 0 0))
   )
@@
     (stroke (width 0) (type default) (color 0 0 0 0))
   )
-  (wire (pts (xy 174.625 83.82) (xy 184.15 83.82))
+  (wire (pts (xy 224.663 143.637) (xy 234.188 143.637))
     (stroke (width 0) (type default) (color 0 0 0 0))
   )
@@
     (stroke (width 0) (type default) (color 0 0 0 0))
   )
-  (wire (pts (xy 174.625 73.025) (xy 183.515 73.025))
+  (wire (pts (xy 224.663 132.842) (xy 233.553 132.842))
     (stroke (width 0) (type default) (color 0 0 0 0))
   )
@@
     (stroke (width 0) (type default) (color 0 0 0 0))
   )
-  (wire (pts (xy 172.72 83.82) (xy 174.625 83.82))
+  (wire (pts (xy 222.758 143.637) (xy 224.663 143.637))
     (stroke (width 0) (type default) (color 0 0 0 0))
   )
@@
     (stroke (width 0) (type default) (color 0 0 0 0))
   )
-  (wire (pts (xy 191.135 73.025) (xy 196.85 73.025))
+  (wire (pts (xy 241.173 132.842) (xy 246.888 132.842))
     (stroke (width 0) (type default) (color 0 0 0 0))
   )
@@
     (stroke (width 0) (type default) (color 0 0 0 0))
   )
-  (wire (pts (xy 174.625 89.535) (xy 174.625 83.82))
+  (wire (pts (xy 224.663 149.352) (xy 224.663 143.637))
     (stroke (width 0) (type default) (color 0 0 0 0))
   )
@@
     (effects (font (size 1.27 1.27)) (justify left bottom))
   )
-  (text "Check this Change once\n" (at 227.33 82.55 0)
-    (effects (font (size 1.27 1.27) (thickness 0.254) bold italic) (justify left bottom))
+  (text "VFB = 0.8V\nVout = (R1/R2 + 1) * VFB" (at 197.612 70.358 0)
+    (effects (font (size 1.27 1.27)) (justify left bottom))
   )
   (text "VFB = 0.85V\nVout = (R1/R2 + 1) * VFB" (at 98.425 172.085 0)
@@
     (effects (font (size 1.27 1.27)) (justify left bottom))
   )
-  (hierarchical_label "MCU_POW" (shape bidirectional) (at 196.85 83.82 0)
+  (hierarchical_label "MCU_POW" (shape bidirectional) (at 246.888 143.637 0)
     (effects (font (size 1.27 1.27)) (justify left))
   )
@@
     (effects (font (size 1.27 1.27)) (justify right))
   )
-  (hierarchical_label "Sun_sensor_power" (shape bidirectional) (at 196.85 89.535 0)
+  (hierarchical_label "Sun_sensor_power" (shape bidirectional) (at 246.888 149.352 0)
     (effects (font (size 1.27 1.27)) (justify left))
   )
-  (hierarchical_label "3V3" (shape bidirectional) (at 158.75 83.82 180)
+  (hierarchical_label "3V3" (shape bidirectional) (at 208.788 143.637 180)
     (effects (font (size 1.27 1.27)) (justify right))
   )
@@
     (effects (font (size 1.27 1.27)) (justify left))
   )
-  (hierarchical_label "Magnetometer_Power" (shape bidirectional) (at 196.85 73.025 0)
+  (hierarchical_label "Magnetometer_Power" (shape bidirectional) (at 246.888 132.842 0)
     (effects (font (size 1.27 1.27)) (justify left))
   )
@@
     (pin "2")
   )
-  (symbol (lib_id "Device:R") (at 187.325 73.025 90) (unit 1)
-    (in_bom yes) (on_board yes) (fields_autoplaced)
-    (property "Reference" "RP6" (id 0) (at 187.325 67.31 90))
-    (property "Value" "0" (id 1) (at 187.325 69.85 90))
-    (property "Footprint" "Resistor_SMD:R_0603_1608Metric" (id 2) (at 187.325 74.803 90)
-      (effects (font (size 1.27 1.27)) hide)
-    )
-    (property "Datasheet" "~" (id 3) (at 187.325 73.025 0)
+  (symbol (lib_id "Device:R") (at 237.363 132.842 90) (unit 1)
+    (in_bom yes) (on_board yes) (fields_autoplaced)
+    (property "Reference" "RP6" (id 0) (at 237.363 127.127 90))
+    (property "Value" "0" (id 1) (at 237.363 129.667 90))
+    (property "Footprint" "Resistor_SMD:R_0603_1608Metric" (id 2) (at 237.363 134.62 90)
+      (effects (font (size 1.27 1.27)) hide)
+    )
+    (property "Datasheet" "~" (id 3) (at 237.363 132.842 0)
       (effects (font (size 1.27 1.27)) hide)
     )
@@
     (pin "1")
   )
-  (symbol (lib_id "Device:R") (at 187.325 89.535 90) (unit 1)
+  (symbol (lib_id "Device:R") (at 237.363 149.352 90) (unit 1)
     (in_bom yes) (on_board yes)
-    (property "Reference" "RP7" (id 0) (at 187.325 92.71 90))
-    (property "Value" "0" (id 1) (at 187.325 86.36 90))
-    (property "Footprint" "Resistor_SMD:R_0603_1608Metric" (id 2) (at 187.325 91.313 90)
-      (effects (font (size 1.27 1.27)) hide)
-    )
-    (property "Datasheet" "~" (id 3) (at 187.325 89.535 0)
+    (property "Reference" "RP7" (id 0) (at 237.363 152.527 90))
+    (property "Value" "0" (id 1) (at 237.363 146.177 90))
+    (property "Footprint" "Resistor_SMD:R_0603_1608Metric" (id 2) (at 237.363 151.13 90)
+      (effects (font (size 1.27 1.27)) hide)
+    )
+    (property "Datasheet" "~" (id 3) (at 237.363 149.352 0)
       (effects (font (size 1.27 1.27)) hide)
     )
@@
     (pin "2")
   )
-  (symbol (lib_id "Device:R") (at 187.96 83.82 90) (unit 1)
+  (symbol (lib_id "Device:R") (at 237.998 143.637 90) (unit 1)
     (in_bom yes) (on_board yes)
-    (property "Reference" "RP8" (id 0) (at 189.865 81.28 90))
-    (property "Value" "0" (id 1) (at 186.055 81.28 90))
-    (property "Footprint" "Resistor_SMD:R_0603_1608Metric" (id 2) (at 187.96 85.598 90)
-      (effects (font (size 1.27 1.27)) hide)
-    )
-    (property "Datasheet" "~" (id 3) (at 187.96 83.82 0)
+    (property "Reference" "RP8" (id 0) (at 239.903 141.097 90))
+    (property "Value" "0" (id 1) (at 236.093 141.097 90))
+    (property "Footprint" "Resistor_SMD:R_0603_1608Metric" (id 2) (at 237.998 145.415 90)
+      (effects (font (size 1.27 1.27)) hide)
+    )
+    (property "Datasheet" "~" (id 3) (at 237.998 143.637 0)
       (effects (font (size 1.27 1.27)) hide)
     )
@@
     (pin "1")
   )
-  (symbol (lib_id "Device:R") (at 168.91 83.82 90) (unit 1)
-    (in_bom yes) (on_board yes) (fields_autoplaced)
-    (property "Reference" "RP5" (id 0) (at 168.91 77.47 90))
-    (property "Value" "0" (id 1) (at 168.91 80.01 90))
-    (property "Footprint" "Resistor_SMD:R_0603_1608Metric" (id 2) (at 168.91 85.598 90)
-      (effects (font (size 1.27 1.27)) hide)
-    )
-    (property "Datasheet" "~" (id 3) (at 168.91 83.82 0)
-      (effects (font (size 1.27 1.27)) hide)
-    )
+  (symbol (lib_id "Device:R") (at 218.948 143.637 90) (unit 1)
+    (in_bom yes) (on_board yes) (fields_autoplaced)
+    (property "Reference" "RP5" (id 0) (at 218.948 137.287 90))
+    (property "Value" "0" (id 1) (at 218.948 139.827 90))
+    (property "Footprint" "Resistor_SMD:R_0603_1608Metric" (id 2) (at 218.948 145.415 90)
+      (effects (font (size 1.27 1.27)) hide)
+    )
+    (property "Datasheet" "~" (id 3) (at 218.948 143.637 0)
+      (effects (font (size 1.27 1.27)) hide)
+    )

Commit message: MCU circuitry forgot LOL
Parts:
- renumbered CP8 to CP1, CP9 to CP3, CP6 to CP4, CP7 to CP5, CP1 to CP6, CP3 to CP7, CP4 to CP8, CP5 to CP9, LP3 to LP1, LP1 to LP2, LP2 to LP3, RP9 to RP1, RP4 to RP10, RP1 to RP2, RP10 to RP3, RP2 to RP4, RP6 to RP5, RP5 to RP6, RP8 to RP7, RP3 to RP8, RP7 to RP9, UP3 to UP1, UP1 to UP2, UP2 to UP3

Commit message: inductor part numbers added
Other:
- note added: "MSS1278H-393MED"
- note added: "XFL4020-332MEB"
Changed lines of the file:
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@@
+    (effects (font (size 1.27 1.27)) (justify left bottom))
+  )
+  (text "MSS1278H-393MED" (at 118.11 119.38 0)
+    (effects (font (size 1.27 1.27)) (justify left bottom))
+  )
+  (text "\n    XFL4020-332MEB" (at 220.98 26.67 0)
+    (effects (font (size 1.27 1.27)) (justify left bottom))
+  )
+  (text "\n    XFL4020-332MEB" (at 102.87 27.94 0)
     (effects (font (size 1.27 1.27)) (justify left bottom))
   )
