File: DRV1.kicad_sch (KiCad schematic)
At the start: 15 parts

Commit message: MCU circuitry forgot LOL
Parts:
- renumbered CA4 to CA1, CA1 to CA2, CA2 to CA3, CA3 to CA4
Changed lines of the file:
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@@
   (symbol (lib_id "pspice:C") (at 124.46 147.32 0) (unit 1)
     (in_bom yes) (on_board yes) (fields_autoplaced)
-    (property "Reference" "CA1" (id 0) (at 129.54 146.0499 0)
+    (property "Reference" "CA2" (id 0) (at 129.54 146.0499 0)
       (effects (font (size 1.27 1.27)) (justify left))
     )
@@
   (symbol (lib_id "upsat-comms-hardware:GND") (at 154.94 154.305 0) (unit 1)
     (in_bom yes) (on_board yes) (fields_autoplaced)
-    (property "Reference" "#PWR011" (id 0) (at 154.94 160.655 0)
+    (property "Reference" "#PWR014" (id 0) (at 154.94 160.655 0)
       (effects (font (size 1.27 1.27)) hide)
     )
@@
   (symbol (lib_id "pspice:C") (at 139.7 147.32 0) (unit 1)
     (in_bom yes) (on_board yes) (fields_autoplaced)
-    (property "Reference" "CA2" (id 0) (at 144.78 146.0499 0)
+    (property "Reference" "CA3" (id 0) (at 144.78 146.0499 0)
       (effects (font (size 1.27 1.27)) (justify left))
     )
@@
   (symbol (lib_id "pspice:C") (at 154.94 147.32 0) (unit 1)
     (in_bom yes) (on_board yes) (fields_autoplaced)
-    (property "Reference" "CA3" (id 0) (at 160.02 146.0499 0)
+    (property "Reference" "CA4" (id 0) (at 160.02 146.0499 0)
       (effects (font (size 1.27 1.27)) (justify left))
     )
@@
   (symbol (lib_id "upsat-comms-hardware:GND") (at 138.43 114.3 0) (unit 1)
     (in_bom yes) (on_board yes) (fields_autoplaced)
-    (property "Reference" "#PWR09" (id 0) (at 138.43 120.65 0)
+    (property "Reference" "#PWR010" (id 0) (at 138.43 120.65 0)
       (effects (font (size 1.27 1.27)) hide)
     )
@@
   (symbol (lib_id "upsat-comms-hardware:GND") (at 153.67 127 0) (unit 1)
     (in_bom yes) (on_board yes) (fields_autoplaced)
-    (property "Reference" "#PWR010" (id 0) (at 153.67 133.35 0)
+    (property "Reference" "#PWR012" (id 0) (at 153.67 133.35 0)
       (effects (font (size 1.27 1.27)) hide)
     )
@@
   (symbol (lib_id "upsat-comms-hardware:GND") (at 222.25 149.86 0) (unit 1)
     (in_bom yes) (on_board yes) (fields_autoplaced)
-    (property "Reference" "#PWR014" (id 0) (at 222.25 156.21 0)
+    (property "Reference" "#PWR013" (id 0) (at 222.25 156.21 0)
       (effects (font (size 1.27 1.27)) hide)
     )
@@
   (symbol (lib_id "upsat-comms-hardware:GND") (at 189.23 119.38 0) (unit 1)
     (in_bom yes) (on_board yes) (fields_autoplaced)
-    (property "Reference" "#PWR012" (id 0) (at 189.23 125.73 0)
+    (property "Reference" "#PWR011" (id 0) (at 189.23 125.73 0)
       (effects (font (size 1.27 1.27)) hide)
     )
@@
   (symbol (lib_id "pspice:C") (at 189.23 113.03 0) (unit 1)
     (in_bom yes) (on_board yes) (fields_autoplaced)
-    (property "Reference" "CA4" (id 0) (at 194.31 111.7599 0)
+    (property "Reference" "CA1" (id 0) (at 194.31 111.7599 0)
       (effects (font (size 1.27 1.27)) (justify left))
     )
@@
   (symbol (lib_id "upsat-comms-hardware:GND") (at 205.74 111.76 0) (unit 1)
     (in_bom yes) (on_board yes) (fields_autoplaced)
-    (property "Reference" "#PWR013" (id 0) (at 205.74 118.11 0)
-      (effects (font (size 1.27 1.27)) hide)
-    )
+    (property "Reference" "#PWR09" (id 0) (at 205.74 118.11 0)
+      (effects (font (size 1.27 1.27)) hide)
+    )

Commit message: All frequency sensitive caps and specific inductor PNs added
Other:
- note added: "0603B105K160XD"
Changed lines of the file:
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@@
     (effects (font (size 1.27 1.27) (thickness 0.254) bold italic) (justify left bottom))
+  )
+  (text "0603B105K160XD" (at 105.41 148.59 0)
+    (effects (font (size 1.27 1.27)) (justify left bottom))
   )
   (label "RTRY" (at 173.355 91.44 180)
